File: Dirty P.sch (EAGLE design)
At the start: 29 parts, among them SW1 FOOT_SW, SW2 108-0020-EVX, U1 MMBT3906, U2 MMBT3906, U3 MMBT3906

Commit message: Rev 3 Complete.
Parts:
- removed EM1: 6-1462037-4, PP_Electromechanical:DPDT_RELAY_IM_RELAY
- added U$2: DB_LOGO_COPPER_MEDIUM, PP_Aesthetics:DB_LOGO_COPPER_MEDIUM
- SW1: value FOOT_SW -> (none); device PP_Electromechanical:SPDT_FOOT_SW -> PP_Electromechanical:3PDT_STOMPBOX_SW
- U$1: REVNUM REV: 2 -> REV: 3
Connections:
- removed net N$21: EM1.POS, SW1.1
- net 9V: no longer SW1.C
- net GND: now also SW1.6
- net N$11: now also SW1.8; no longer EM1.3
- net N$14: now also SW1.1, SW1.5; no longer EM1.5
- net N$17: now also SW1.3, SW1.9; no longer EM1.2, EM1.7
- net N$19: now also SW1.7; no longer EM1.4
- net N$4: no longer EM1.NEG
- net SIG_IN: now also SW1.2; no longer EM1.6
Other:
- moved on the sheet: BATT1
